File: hardware/g1-sd-wifi/controller/KUI-G1-Bridge-RevA.kicad_sch (KiCad schematic)
At the start: 39 parts, among them J1 10103594-0001LF, J2 TSW-126-07-L-D, J3 TSW-126-07-L-D, J4 SM03B-SRSS-TB(LF)(SN), SW1 434133025816, SW2 434133025816, U1 RP2350B, U2 NCP1117ST33T3G, U3 W25Q128JVSIQ, X1 12MHz

Commit message: Implement G1 bridge circuit and flex; add carrier routing checkpoint
Add the native RP2350B/MachXO2/C5 circuit, optional 8 MiB PSRAM assembly variant, raw G1 probes, USB-free C5 recovery and optional independent stock BIOS recovery. Implement tested default-off FPGA activation and shared diagnostic receipt, exact catalog part identities, two routed CN503 flex arms, native assembly candidates and actual-size fit PDFs.

Both flex boards pass ERC/DRC/parity. Static circuit integration checks 1204 assigned endpoints and 8240 safety cases. FPGA simulations and resource mapping pass; device timing and firmware remain pending. Independent carrier checks confirm all 16 manufacturer C5 contact positions, all 40 flex mating positions, continuous ground contour and zero native geometry/parity violations.

This carrier checkpoint has 600 uncapped open connections. Complete routing, secondary bypass layout, installed fit/support and assembly/supplier agreement remain open. The fabrication exporter stays blocked and no order archives are released.
Parts:
- removed C1, C19, C5: 10u, RPI_COMPILED:generic_capc2012x125, symbol KUI_RP_Reference:RPI_DB__Capacitors | MLCC | M2012/RP-01GYSK-AVBE41
- removed C10, C11, C12, C13, C14, C15, C16, C17, C18, C2, C20, C21, C8: 100n, RPI_COMPILED:generic_capc1005x50, symbol KUI_RP_Reference:RPI_DB__Capacitors | MLCC | M1005/RP-01BJ9Y-KRGF41
- removed C3, C4: 15p, RPI_COMPILED:generic_capc1005x50, symbol KUI_RP_Reference:RPI_DB__Capacitors | MLCC | M1005/RP-01C89W-LLY9XV
- removed C6, C7: 4.7u, RPI_COMPILED:generic_capc1005x50_wide, symbol KUI_RP_Reference:RPI_DB__Capacitors | MLCC | M1005/RP-019A1P-0C2GHY
- removed C9: 4.7u, RPI_COMPILED:generic_capc1005x50, symbol KUI_RP_Reference:RPI_DB__Capacitors | MLCC | M1005/RP-019A1P-0C2GHY
- removed J1: 10103594-0001LF, RPI_COMPILED:amphenol_10103594-0001lf, symbol KUI_RP_Reference:RPI_DB__Connectors | USB/RP-019A1P-1JAX7V
- removed J2, J3: TSW-126-07-L-D, RPI_COMPILED:samtec_tsw-126-07-l-d, symbol KUI_RP_Reference:RPI_DB__Connectors | Pin_Headers/RP-01KJ62-FD8Y6K
- removed J4: SM03B-SRSS-TB(LF)(SN), RPI_COMPILED:jst_sm03b-srss-tb-lf--sn-, symbol KUI_RP_Reference:RPI_DB__Connectors | Rectangular/RP-01EKJ1-8V9SV1
- removed L1: 3.3u, RPI_COMPILED:abracon_aota-b201610s3r3-101-t, symbol KUI_RP_Reference:RPI_DB__Inductors | Fixed | M2016/RP-01GY5D-2VC7WP
- removed R10: 0, RPI_COMPILED:generic_resc1005x35, symbol KUI_RP_Reference:RPI_DB__Resistors | Chip | M1005/RP-019A1P-4Y4V63
- removed R2, R4, R6: 1k, RPI_COMPILED:generic_resc1005x35, symbol KUI_RP_Reference:RPI_DB__Resistors | Chip | M1005/RP-019A1P-4Z6ZWY
- removed R3: 33, RPI_COMPILED:generic_resc1005x35, symbol KUI_RP_Reference:RPI_DB__Resistors | Chip | M1005/RP-019A1P-58PW9L
- removed R7, R8: 27, RPI_COMPILED:generic_resc1005x35, symbol KUI_RP_Reference:RPI_DB__Resistors | Chip | M1005/RP-01C89V-LTEYC4
- removed SW1, SW2: 434133025816, RPI_COMPILED:wurthelek_434133025816, symbol KUI_RP_Reference:RPI_DB__Electromechanical | Switches | Tactile/RP-01H0MT-6E9H8F
- removed U1: RP2350B, RPI_COMPILED:rpi_rp2350b_vias, symbol KUI_RP_Reference:RPI_DB__Integrated_Circuits | Microcontrollers/RP-01HA9H-ABBLJN
- removed U2: NCP1117ST33T3G, RPI_COMPILED:onsemi_ncp1117st33t3g, symbol KUI_RP_Reference:RPI_DB__Integrated_Circuits | Power | LDO/RP-01JWD9-7JRX6J
- removed U3: W25Q128JVSIQ, RPI_COMPILED:generic_soic127p790x195-8, symbol KUI_RP_Reference:RPI_DB__Integrated_Circuits | Memory | Serial_Flash | SPI/RP-0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
- removed X1: 12MHz, RPI_COMPILED:generic_xtalcc320x250x80-4, symbol KUI_RP_Reference:RPI_DB__Frequency_Timing | Crystals/RP-01G8X7-GS352B
Connections:
- no-connect marks 1 -> 0
Other:
- added sheet bios-1 (bios-1.kicad_sch)
- added sheet cn503-interface-1 (cn503-interface-1.kicad_sch)
- added sheet controller-1 (controller-1.kicad_sch)
- added sheet controller-2 (controller-2.kicad_sch)
- added sheet controller-3 (controller-3.kicad_sch)
- added sheet frontend-1 (frontend-1.kicad_sch)
- added sheet frontend-2 (frontend-2.kicad_sch)
- added sheet power-bus-1 (power-bus-1.kicad_sch)
- added sheet power-bus-2 (power-bus-2.kicad_sch)
- added sheet power-bus-3 (power-bus-3.kicad_sch)
- added sheet power-source-declarations-1 (power-source-declarations-1.kicad_sch)
- note added: "Retained GD-ROM device 0 / bridge device 1. Original mask ROM recovery is a hardware path. 8 MiB PSRAM is bridge cache. Native 4-bit SD exposes raw sectors to K-UI. Review source contracts and validation reports; prototype qualification remains open."
- note removed: "12MHz Crystal"
- note removed: "BENCH GPIO BREAKOUTS ONLY Not a Dreamcast GD-ROM connector pinout."
- note removed: "BOOTSEL Button"
- note removed: "CONTROLLER FOUNDATION - DRAFT MCU-side signal allocation only. G1 buffers and bus isolation pending. J2/J3 are bench GPIO breakouts; they are not the GD-ROM pad map. MicroSD and XIAO circuits pending. USB bench power only; Dreamcast power, hold-up and USB isolation pending. RP2350B must use A4 stepping. NOT READY FOR FABRICATION."
- note removed: "IOs"
- note removed: "JST Debug Connector"
- note removed: "MAINBOARD ATTACHMENT / UNDERSIDE MOUNT VA1 solder-pad mapping; no drive PCB identity needed. Vertical clearance, shield gap and XIAO socket height pending."
- note removed: "Make sure R7 and R8 are close to RP2350"
- note removed: "POWER REQUIREMENTS - CIRCUIT PENDING 3.3 V G1 logic. Core/SD: 3.3 V input or regulated 5 V input. C5: separate switched 5 V feed; 3.3 V-only mode needs boost. USB isolation and SD/core hold-up still require design."
- note removed: "Power"
- note removed: "Primary Flash"
- note removed: "RUN Button"
- note removed: "Secondary Flash/PSRAM"
- note removed: "USB BENCH POWER - power architecture pending"
- company: K-UI -> K-UI NeXT
- title: K-UI G1 Bridge - Controller Foundation -> G1 microSD / Wi-Fi bridge — Rev A circuit implementation
