File: hardware/g1-sd-wifi/controller/bios-1.kicad_sch (KiCad schematic)
At the start: 33 parts, among them J40 FH12-14S-0.5SH(55), J41 FH12-6S-0.5SH(55), SW40 STOCK_RECOVERY / CUSTOM (OFFB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, U40 MX29LV640ETTI-70G x8 / 4 x 2M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, U41 SN74LVC2G125 bank-domain buff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, U42 SN74LVC1G11 write-authorize A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, U43 SN74LVC1G04 write-block inver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, U44 SN74LVC1G332 NOR WE qualifier, U45 TLV803EB29 console-rail NOR r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

Commit message: G1 carrier: 1k R410, 4.18 V loss threshold, local bypass placement
- R410 becomes a 1 kOhm pull-up (reused 0402 part), so a selector harness
  fitted with R410 still present cannot short console 3.3 V.
- R270 (4.7 kOhm, reused part) lowers the U26 loss threshold from 4.358 V
  to 4.180 V; the divider now sits beside U26 instead of 27 mm away.
- 28 owner-assigned bypass capacitors placed next to their ICs with a new
  placer (tools/place_local_bypass.py); C230 and the DNP BIOS caps for
  U42/U43 remain open. C236 moves to the C5 load.
- tools/update_board_from_netlist.py applies reviewed schematic changes to
  the routed board without re-placing it.
- generate_design.py takes KICAD10_FOOTPRINT_DIR so an older system library
  cannot overwrite the localized KiCad 10 footprints.

Native ERC 0, DRC 0, parity 0; integration audit refreshed and passing.

Co-Authored-By: Claude Opus 5.5 <noreply@anthropic.com>
Claude-Session: https://claude.ai/code/session_01Gp9EYc2r9fMpZ7V8WtfonZ
Parts:
- R410: value 0R -> 1k; footprint KUI_Footprints:R_0603_1608Metric -> KUI_Footprints:R_0402_1005Metric; MPN RC0603JR-070RL -> RC0402FR-071KL
Changed lines of the file:
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@@
 (symbol (lib_id "KUI_G1:R410") (at 259.08 110.49 0) (unit 1) (in_bom yes) (on_board yes) (dnp no)
  (property "Reference" "R410" (at 259.08 102.87 0) (effects (font (size 1.0 1.0))))
- (property "Value" "0R" (at 259.08 105.41 0) (effects (font (size 1.0 1.0))))
- (property "Footprint" "KUI_Footprints:R_0603_1608Metric" (at 259.08 110.49 0) (effects (font (size 1.0 1.0)) hide))
+ (property "Value" "1k" (at 259.08 105.41 0) (effects (font (size 1.0 1.0))))
+ (property "Footprint" "KUI_Footprints:R_0402_1005Metric" (at 259.08 110.49 0) (effects (font (size 1.0 1.0)) hide))
  (property "Datasheet" "" (at 259.08 110.49 0) (effects (font (size 1.0 1.0)) hide))
- (property "MPN" "RC0603JR-070RL" (at 259.08 110.49 0) (effects (font (size 1.0 1.0)) hide))
+ (property "MPN" "RC0402FR-071KL" (at 259.08 110.49 0) (effects (font (size 1.0 1.0)) hide))
  (property "LCSC" "" (at 259.08 110.49 0) (effects (font (size 1.0 1.0)) hide))
  (property "Variant" "BASE_ONLY" (at 259.08 110.49 0) (effects (font (size 1.0 1.0)) hide))
