File: hardware/g1-sd-wifi/controller/frontend-1.kicad_sch (KiCad schematic)
At the start: 45 parts, among them J10 FPGA JTAG pogo pads, U10 LCMXO2-2000HC-4TG100C, X10 50MHz 3.3V

Commit message: G1 carrier: re-floorplan around the FPGA on six layers (unrouted)
The four-layer placement stalled the router at 300+ open connections.
Pin plan and floorplan were the cause, not just layer count:

- FPGA pins follow the placement (design/fpga-pin-swap-2026-10-10.json):
  the RP2350 link bus moves to the east edge facing the controller (it
  was on the west edge, wrapping round the chip), BUS_DD to the south
  edge in U35's A-side order, host controls/requests/BIOS lines to the
  west edge, the 50 MHz clock to PCLKT5_0 (pin 3). Only FPGA_CLK50 is a
  clock in the RTL; all other moves are plain LVCMOS33 I/O. LPF and pin
  table regenerate from frontend.json via tools/sync_fpga_pins.py.
- U35 turns +90 degrees and sits directly under the FPGA (which moves
  2.26 mm north), so the data bus drops straight between them.
- The 16 raw ATA_DD probes and their ground probe move from U35 (whose
  B side now faces the BIOS aperture) to U40's pins on the same nets.
- Small ICs, bypass capacitors and passives are re-placed by
  connectivity; narrow plane fanout regenerated; six-layer stack
  (F / GND / sig / sig / +3V3 / B, 0.8 mm).

tools/floorplan_2026_10_10.sh reproduces the board from the previous
commit. ERC 0, schematic parity 0, native DRC 0 violations; integration
audit and FPGA checks pass. Routing is in progress.

Co-Authored-By: Claude Opus 5.5 <noreply@anthropic.com>
Claude-Session: https://claude.ai/code/session_01Gp9EYc2r9fMpZ7V8WtfonZ
Connections:
- net BIOS_BANK0: now also U10.7 (PL4A); no longer U10.78 (PT22A)
- net BIOS_BANK1: now also U10.4 (PL3B); no longer U10.83 (PT19B)
- net BIOS_RECOVERYn: now also U10.19 (PL11B); no longer U10.96 (PT11B)
- net BIOS_WR_EN: now also U10.20 (PL12A); no longer U10.84 (PT19A)
- net BRIDGE_ARM: now also U10.58 (PR11A); no longer U10.21 (PL12B)
- net BUS_CS0n: now also U10.12 (PL7C); no longer U10.34 (PB11A)
- net BUS_CS1n: now also U10.13 (PL7D); no longer U10.35 (PB11B)
- net BUS_DA0: now also U10.8 (PL4B); no longer U10.28 (PB5B)
- net BUS_DA1: now also U10.9 (PL5A); no longer U10.29 (PB6A)
- net BUS_DA2: now also U10.10 (PL5B); no longer U10.30 (PB6B)
- net BUS_DD0: now also U10.28 (PB5B); no longer U10.51 (PR14B)
- net BUS_DD1: now also U10.29 (PB6A); no longer U10.52 (PR14A)
- net BUS_DD10: now also U10.41 (PB18B); no longer U10.63 (PR7A)
- net BUS_DD11: now also U10.42 (PB21A); no longer U10.64 (PR6B)
- net BUS_DD12: now also U10.43 (PB21B); no longer U10.65 (PR6A)
- net BUS_DD13: now also U10.45 (PB22A); no longer U10.66 (PR5B)
- net BUS_DD14: now also U10.47 (PB22B); no longer U10.67 (PR5A)
- net BUS_DD15: now also U10.51 (PR14B); no longer U10.68 (PR4B)
- net BUS_DD2: now also U10.30 (PB6B); no longer U10.53 (PR12B)
- net BUS_DD3: now also U10.34 (PB11A); no longer U10.54 (PR12A)
- net BUS_DD4: now also U10.35 (PB11B); no longer U10.57 (PR11B)
- net BUS_DD5: now also U10.36 (PB12A); no longer U10.58 (PR11A)
- net BUS_DD6: now also U10.37 (PB12B); no longer U10.59 (PR10B)
- net BUS_DD7: now also U10.38 (PB16A); no longer U10.60 (PR10A)
- net BUS_DD8: now also U10.39 (PB16B); no longer U10.61 (PR9A)
- net BUS_DD9: now also U10.40 (PB18A); no longer U10.62 (PR7B)
- net BUS_DIORn: now also U10.14 (PL9A); no longer U10.36 (PB12A)
- net BUS_DIOWn: now also U10.15 (PL9B); no longer U10.37 (PB12B)
- net BUS_DMACKn: now also U10.16 (PL10A); no longer U10.39 (PB16B)
- net BUS_RESETn: now also U10.17 (PL10B); no longer U10.38 (PB16A)
- net BUS_SAFE: now also U10.25 (PL14B); no longer U10.24 (PL14A)
- net DATA_DIR: now also U10.54 (PR12A); no longer U10.70 (PR3B)
- net FPGA_CLK50: now also U10.3 (PL3A); no longer U10.20 (PL12A)
- net FPGA_READY: now also U10.52 (PR14A); no longer U10.97 (PT11A)
- net FPGA_RESETn: now also U10.59 (PR10B); no longer U10.19 (PL11B)
- net LINK_A0: now also U10.63 (PR7A); no longer U10.15 (PL9B)
- net LINK_A1: now also U10.62 (PR7B); no longer U10.16 (PL10A)
- net LINK_D0: now also U10.75 (PR1A); no longer U10.1 (PL2A)
- net LINK_D1: now also U10.74 (PR1B); no longer U10.2 (PL2B)
- net LINK_D2: now also U10.71 (PR3A); no longer U10.4 (PL3B)
- net LINK_D3: now also U10.70 (PR3B); no longer U10.7 (PL4A)
- net LINK_D4: now also U10.69 (PR4A); no longer U10.8 (PL4B)
- net LINK_D5: now also U10.68 (PR4B); no longer U10.9 (PL5A)
- net LINK_D6: now also U10.67 (PR5A); no longer U10.10 (PL5B)
- net LINK_D7: now also U10.66 (PR5B); no longer U10.12 (PL7C)
- net LINK_IRQ: now also U10.61 (PR9A); no longer U10.17 (PL10B)
- net LINK_RDn: now also U10.64 (PR6B); no longer U10.14 (PL9A)
- net LINK_READY: now also U10.60 (PR10A); no longer U10.18 (PL11A)
- net LINK_WRn: now also U10.65 (PR6A); no longer U10.13 (PL7D)
- net PWR_FAILn: now also U10.57 (PR11B); no longer U10.25 (PL14B)
- net REQ_DATA_OEn: now also U10.53 (PR12B); no longer U10.69 (PR4A)
- net REQ_DMARQ: now also U10.21 (PL12B); no longer U10.75 (PR1A)
- net REQ_DMARQ_OEn: now also U10.1 (PL2A); no longer U10.41 (PB18B)
- net REQ_INTRQ: now also U10.18 (PL11A); no longer U10.74 (PR1B)
- net REQ_INTRQ_OEn: now also U10.2 (PL2B); no longer U10.40 (PB18A)
- net REQ_IORDY_LOW: now also U10.24 (PL14A); no longer U10.71 (PR3A)
