File: hardware/g1-sd-wifi/controller/power-bus-2.kicad_sch (KiCad schematic)
At the start: 51 parts, among them U31 SN74LVC2G04DBVT, U32 SN74LVC1G32DBVR, U33 SN74LVC1G08DBVR, U34 SN74LVC1G08DBVR

Commit message: G1 carrier: FPGA pull-downs replace the sixteen BUS_DD biases
The 47 k biases on BUS_DD (between the FPGA and U35's A port) found no
room near that bus and were placed up to 40 mm away; their connections
were a quarter of what the router could not close. The FPGA's own I/O
pull-down now holds BUS_DD during tri-state idle (PULLMODE=DOWN in the
LPF, emitted by sync_fpga_pins.py). Before configuration U35 is held
disabled by its DATA_OEn pull-up; the MachXO2's unconfigured pin state
is to be confirmed against Lattice TN1202 at bring-up. The host-side
ATA_DD biases stay.

- power-bus.json drops R223..R253 (odd); integration counts 349/360/351;
  ERC 0; integration audit passes; parts list BASE 263 fitted parts.
- update_board_from_netlist: --allow-remove deletes a removed part's
  footprint and pad copper.
- floorplan script: removes the biases and places the optional reserve
  bank (C202-C205) beside U20, which it feeds, instead of 90 mm away.
- Board regenerated: 153/153 placed, native DRC 0, parity 0. Routing in
  progress.

Co-Authored-By: Claude Opus 5.5 <noreply@anthropic.com>
Claude-Session: https://claude.ai/code/session_01Gp9EYc2r9fMpZ7V8WtfonZ
Parts:
- removed R223: 47k, KUI_Footprints:R_0402_1005Metric, symbol KUI_G1:R223
- removed R225: 47k, KUI_Footprints:R_0402_1005Metric, symbol KUI_G1:R225
- removed R227: 47k, KUI_Footprints:R_0402_1005Metric, symbol KUI_G1:R227
- removed R229: 47k, KUI_Footprints:R_0402_1005Metric, symbol KUI_G1:R229
- removed R231: 47k, KUI_Footprints:R_0402_1005Metric, symbol KUI_G1:R231
- removed R233: 47k, KUI_Footprints:R_0402_1005Metric, symbol KUI_G1:R233
- removed R235: 47k, KUI_Footprints:R_0402_1005Metric, symbol KUI_G1:R235
- removed R237: 47k, KUI_Footprints:R_0402_1005Metric, symbol KUI_G1:R237
- removed R239: 47k, KUI_Footprints:R_0402_1005Metric, symbol KUI_G1:R239
- removed R241: 47k, KUI_Footprints:R_0402_1005Metric, symbol KUI_G1:R241
- removed R243: 47k, KUI_Footprints:R_0402_1005Metric, symbol KUI_G1:R243
- removed R245: 47k, KUI_Footprints:R_0402_1005Metric, symbol KUI_G1:R245
- removed R247: 47k, KUI_Footprints:R_0402_1005Metric, symbol KUI_G1:R247
- removed R249: 47k, KUI_Footprints:R_0402_1005Metric, symbol KUI_G1:R249
- removed R251: 47k, KUI_Footprints:R_0402_1005Metric, symbol KUI_G1:R251
- removed R253: 47k, KUI_Footprints:R_0402_1005Metric, symbol KUI_G1:R253
- added C224: 100nF, KUI_Footprints:C_0402_1005Metric, symbol KUI_G1:C224
- added C225: 100nF, KUI_Footprints:C_0402_1005Metric, symbol KUI_G1:C225
- added C226: 100nF, KUI_Footprints:C_0402_1005Metric, symbol KUI_G1:C226
- added C227: 100nF, KUI_Footprints:C_0402_1005Metric, symbol KUI_G1:C227
- added R254: 47k, KUI_Footprints:R_0402_1005Metric, symbol KUI_G1:R254
- added R255: 47k, KUI_Footprints:R_0402_1005Metric, symbol KUI_G1:R255
- added R256: 47k, KUI_Footprints:R_0402_1005Metric, symbol KUI_G1:R256
- added R257: 47k, KUI_Footprints:R_0402_1005Metric, symbol KUI_G1:R257
- added R258: 47k, KUI_Footprints:R_0402_1005Metric, symbol KUI_G1:R258
- added R259: 47k, KUI_Footprints:R_0402_1005Metric, symbol KUI_G1:R259
- added R260: 47k, KUI_Footprints:R_0402_1005Metric, symbol KUI_G1:R260
- added R261: 47k, KUI_Footprints:R_0402_1005Metric, symbol KUI_G1:R261
- added U35: SN74LVC16T245, KUI_Footprints:TSSOP-48_6.1x12.5mm_P0.5mm, symbol KUI_G1:U35
Connections:
- net +3V3_LOGIC: now also C224.1, C225.1, U35.31 (VCCA), U35.42 (VCCA)
- net ATA_DD0: now also U35.2 (1B1)
- net ATA_DD1: now also U35.3 (1B2)
- net ATA_DD10: now also U35.16 (2B3)
- net ATA_DD11: now also U35.17 (2B4)
- net ATA_DD12: now also U35.19 (2B5)
- net ATA_DD13: now also U35.20 (2B6)
- net ATA_DD14: now also U35.22 (2B7)
- net ATA_DD2: now also U35.5 (1B3)
- net ATA_DD3: now also U35.6 (1B4)
- net ATA_DD4: now also U35.8 (1B5)
- net ATA_DD5: now also U35.9 (1B6)
- net ATA_DD6: now also U35.11 (1B7)
- net ATA_DD7: now also U35.12 (1B8)
- net ATA_DD8: now also U35.13 (2B1)
- net ATA_DD9: now also U35.14 (2B2)
- net BUS_DD0: now also U35.47 (1A1)
- net BUS_DD1: now also U35.46 (1A2)
- net BUS_DD10: now also U35.33 (2A3)
- net BUS_DD11: now also U35.32 (2A4)
- net BUS_DD12: now also U35.30 (2A5)
- net BUS_DD13: now also U35.29 (2A6)
- net BUS_DD14: now also U35.27 (2A7)
- net BUS_DD15: now also U35.26 (2A8)
- net BUS_DD2: now also U35.44 (1A3)
- net BUS_DD3: now also U35.43 (1A4)
- net BUS_DD4: now also U35.41 (1A5)
- net BUS_DD5: now also U35.40 (1A6)
- net BUS_DD6: now also U35.38 (1A7)
- net BUS_DD7: now also U35.37 (1A8)
- net BUS_DD8: now also U35.36 (2A1)
- net BUS_DD9: now also U35.35 (2A2)
- net CONSOLE_3V3: now also C226.1, C227.1, R258.1, R259.1, R260.1, R261.1, U35.18 (VCCB), U35.7 (VCCB)
- net DATA_DIR: now also U35.1 (1DIR), U35.24 (2DIR)
- net DATA_OEn: now also U35.25 (2OEn), U35.48 (1OEn)
- net GND: now also C224.2, C225.2, C226.2, C227.2, R254.2, R255.1, R256.1, R257.1, U35.10 (GND), U35.15 (GND), U35.21 (GND), U35.28 (GND), U35.34 (GND), U35.39 (GND), U35.4 (GND), U35.45 (GND)
- new net ATA_CS0n: R258.2
- new net ATA_CS1n: R259.2
- new net ATA_DA0: R255.2
- new net ATA_DA1: R256.2
- new net ATA_DA2: R257.2
- new net ATA_DD15: R254.1, U35.23 (2B8)
- new net ATA_DIORn: R260.2
- new net ATA_DIOWn: R261.2
Other:
- moved on the sheet: R224, R226, R228, R230, R232, R234, R236, R238, R240, R242, R244, R246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

Commit message: G1 carrier: D21 input TVS turns a 12-V mis-wire into a blown F20
A bidirectional 5-V TVS (SMF5.0CA, SOD-123FL) from FUSED_5V to GND,
between F20 and Q20: above about 6.4 V it conducts far more than F20's
1.5 A rating, so a wrong 12-V feed opens the fuse instead of sitting on
the 5-V parts. Bidirectional, so a reversed 5-V feed stays below
breakdown and Q20 blocks it without blowing F20. Downstream parts may
still see the ~9 V clamp while F20 clears; the doc says so.

Schematic, netlist, ERC (0), integration audit (361 parts) and parts
list regenerated. Its datasheet and JLC catalog identity could not be
reached from this environment, so the part is listed sourcing-pending.
The floorplan places D21 2.2 mm from F20's output; the netlist updater
can now add a part whose footprint is not on the board yet. The power
doc also notes that F20 does not protect the harness itself.

Co-Authored-By: Claude Opus 5.5 <noreply@anthropic.com>
Claude-Session: https://claude.ai/code/session_01Gp9EYc2r9fMpZ7V8WtfonZ
Parts:
- removed R261: 47k, KUI_Footprints:R_0402_1005Metric, symbol KUI_G1:R261
- added C219: 100nF, KUI_Footprints:C_0402_1005Metric, symbol KUI_G1:C219
Connections:
- net +3V3_LOGIC: now also C219.1
- net GND: now also C219.2
Other:
- moved on the sheet: C220, C221, C222, C223, C224, C225, C226, C227, R211, R212, R213, R214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

Commit message: G1 safety: fuse the host 3.3-V entry; no console 5 V on the flex or carrier
Host 3.3 V reached about 30 carrier parts straight from two flex contacts,
and the two console-5-V contacts were joined by an unused carrier trace;
a short on either would load a console supply through 0.5 A connector
contacts with no fuse anywhere. Now:

- F21 (0467.500NR, 0.5 A fast, same 467 family as F20) sits between the one
  remaining 3.3-V entry, J51 B1, and CONSOLE_3V3. If it opens the buffers
  lose VCCB and isolate, and U25 reports the host rail absent.
- CN503 A1 (second 3.3 V) and A3/B3 (5 V) get no flex copper at all: no
  landing pad, no trace, only an unconnected mating finger, so a chafed
  flex cannot short a console supply. Their carrier socket pins are bare.
  flex-interface.json lists them; the flex and carrier generators and both
  checks read that list. Flex ERC/DRC/parity 0; carrier ERC 0, integration
  check pass (362 parts).
- The DSN export keeps the 5-V and storage supply nets on the 1 oz outer
  layers: on 0.5 oz inner copper a 0.25 mm track at the fuse current would
  overheat (IPC-2221).
- F21 is placed by the floorplan next to J51; board DRC 0, parity 0
  (unrouted).

Co-Authored-By: Claude Opus 5.5 <noreply@anthropic.com>
Claude-Session: https://claude.ai/code/session_01Gp9EYc2r9fMpZ7V8WtfonZ
Parts:
- removed R260: 47k, KUI_Footprints:R_0402_1005Metric, symbol KUI_G1:R260
- added U30: SN74LVC1G11DBVR, KUI_Footprints:SOT-23-6, symbol KUI_G1:U30
Connections:
- net +3V3_LOGIC: now also U30.5 (VCC)
- net BUS_SAFE: now also U30.4 (Y)
- net GND: now also U30.2 (GND)
- new net FPGA_ARMED: U30.3 (B)
- new net PWR_GOOD: U30.1 (A)
- new net RESET_RECOVERY_OK: U30.6 (C)
Other:
- moved on the sheet: C219, C220, C221, C222, C223, C224, C225, C226, C227, R211, R212, R213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
