File: hardware/g1-sd-wifi/controller/power-bus-1.kicad_sch (KiCad schematic)
At the start: 49 parts, among them J20 5V/GND direct wire pads, Q20 PMV48XP reverse polarity, U20 TPS2116 automatic mux, U21 TPS62162 3.3V 1A, U22 TPS62162 3.3V 1A, U23 TPS3808G33DBVR, U24 TPS3808G33DBVR, U25 TPS3808G33DBVR, U26 TPS3808G01DBVR, U27 SN74LVC2G08DCUR, U28 SN74LVC2G08DCUR, U29 SN74LVC2G08DCUR

Commit message: Fix G1 protection lands and refresh ordering review
Resolve D21/F21 sourcing and manufacturer-recommended pads; retain Claude's complete routing while widening existing supply paths. Correct local-fault and via-current screening, record remaining qualification, and refresh BOM/CPL, actual-size fit PDFs and review-only artwork.

Native KiCad10.0.7 ERC/DRC/opens/parity0; static integration and normal-current screen pass. Selected fault screen and physical/supplier release conditions remain explicit.
Parts:
- D21: footprint KUI_Footprints:D_SOD-123F -> KUI_Footprints:HighDiode_SMF_SOD123FL; LCSC (none) -> C22458622
- F20: footprint KUI_Footprints:Fuse_0603_1608Metric -> KUI_Footprints:Littelfuse_467_0603_Recommended
- F21: footprint KUI_Footprints:Fuse_0603_1608Metric -> KUI_Footprints:Littelfuse_467_0603_Recommended; LCSC (none) -> C206990
Changed lines of the file:
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@@
  (property "Reference" "F20" (at 55.88 49.53 0) (effects (font (size 1.0 1.0))))
  (property "Value" "1.5A fast fuse" (at 55.88 52.07 0) (effects (font (size 1.0 1.0))))
- (property "Footprint" "KUI_Footprints:Fuse_0603_1608Metric" (at 55.88 57.15 0) (effects (font (size 1.0 1.0)) hide))
+ (property "Footprint" "KUI_Footprints:Littelfuse_467_0603_Recommended" (at 55.88 57.15 0) (effects (font (size 1.0 1.0)) hide))
  (property "Datasheet" "https://www.littelfuse.com/assetdocs/fuse-467-datasheet?assetguid=4a59f034-1cca-460e-a5ba-e1e66247c76d" (at 55.88 57.15 0) (effects (font (size 1.0 1.0)) hide))
  (property "MPN" "046701.5NR" (at 55.88 57.15 0) (effects (font (size 1.0 1.0)) hide))
@@
  (property "Reference" "D21" (at 55.88 87.63 0) (effects (font (size 1.0 1.0))))
  (property "Value" "5 V bidirectional TVS" (at 55.88 90.17 0) (effects (font (size 1.0 1.0))))
- (property "Footprint" "KUI_Footprints:D_SOD-123F" (at 55.88 95.25 0) (effects (font (size 1.0 1.0)) hide))
- (property "Datasheet" "https://www.littelfuse.com/products/overvoltage-protection/tvs-diodes/surface-mount/smf" (at 55.88 95.25 0) (effects (font (size 1.0 1.0)) hide))
+ (property "Footprint" "KUI_Footprints:HighDiode_SMF_SOD123FL" (at 55.88 95.25 0) (effects (font (size 1.0 1.0)) hide))
+ (property "Datasheet" "https://datasheet.lcsc.com/datasheet/pdf/d7261141784d0c4389ea587ce555a8ce.pdf?productCode=C22458622" (at 55.88 95.25 0) (effects (font (size 1.0 1.0)) hide))
  (property "MPN" "SMF5.0CA" (at 55.88 95.25 0) (effects (font (size 1.0 1.0)) hide))
- (property "LCSC" "" (at 55.88 95.25 0) (effects (font (size 1.0 1.0)) hide))
+ (property "LCSC" "C22458622" (at 55.88 95.25 0) (effects (font (size 1.0 1.0)) hide))
  (property "Variant" "BASE" (at 55.88 95.25 0) (effects (font (size 1.0 1.0)) hide))
  (pin "1")
@@
  (property "Reference" "F21" (at 55.88 105.41 0) (effects (font (size 1.0 1.0))))
  (property "Value" "0.5A fast fuse" (at 55.88 107.95 0) (effects (font (size 1.0 1.0))))
- (property "Footprint" "KUI_Footprints:Fuse_0603_1608Metric" (at 55.88 113.03 0) (effects (font (size 1.0 1.0)) hide))
+ (property "Footprint" "KUI_Footprints:Littelfuse_467_0603_Recommended" (at 55.88 113.03 0) (effects (font (size 1.0 1.0)) hide))
  (property "Datasheet" "https://www.littelfuse.com/assetdocs/fuse-467-datasheet?assetguid=4a59f034-1cca-460e-a5ba-e1e66247c76d" (at 55.88 113.03 0) (effects (font (size 1.0 1.0)) hide))
  (property "MPN" "0467.500NR" (at 55.88 113.03 0) (effects (font (size 1.0 1.0)) hide))
- (property "LCSC" "" (at 55.88 113.03 0) (effects (font (size 1.0 1.0)) hide))
+ (property "LCSC" "C206990" (at 55.88 113.03 0) (effects (font (size 1.0 1.0)) hide))
  (property "Variant" "BASE" (at 55.88 113.03 0) (effects (font (size 1.0 1.0)) hide))
  (pin "1")
