File: hardware/g1-sd-wifi/controller/power-bus-1.kicad_sch (KiCad schematic)
At the start: 49 parts, among them J20 5V/GND direct wire pads, Q20 PMV48XP reverse polarity, U20 TPS2116 automatic mux, U21 TPS62162 3.3V 1A, U22 TPS62162 3.3V 1A, U23 TPS3808G33DBVR, U24 TPS3808G33DBVR, U25 TPS3808G33DBVR, U26 TPS3808G01DBVR, U27 SN74LVC2G08DCUR, U28 SN74LVC2G08DCUR, U29 SN74LVC2G08DCUR

Commit message: G1 readiness: close the converter fault screen, measurement plan with pass numbers
Converters: U21/U22 become TPS62172DSGR (0.5 A, static high-side limit
1.35 A max) instead of TPS62162DSGR (2.45 A max); same DSG0008A pinout and
FB = AGND. Three 0.15 mm +3V3_LOGIC links beside R2038 are widened to
0.20 mm in place. check_power_copper.py screens the converters at the exact
1.35 A and passes with no failures (the 2.5 A screen of the old part had
138). tools/power_fault_screen_2026_10_23.sh replays it from 6d50fc5:
DRC/opens/parity 0, the power screen gate, and check_preservation.py (new
--allow-change, which accepts only a track width or a text string, with
the text's position and size still compared) shows only the three widths
and a corrected Dwgs.User note changed. The pass has 2.7 % margin on the
87 single logic plane-to-pad vias; that is recorded. LCSC C59873
comes from a search index and is listed for the owner to confirm.

Readiness review: the flex sockets J50/J51 must move before either order
(arm B cannot reach J51 as placed); this is documented as the next layout
revision, to follow the owner's fit check and a new flex route survey.
docs/OWNER-NEXT-STEPS.md is rewritten so every measurement has a pass
number (CN503 row and numbering proof with negative pairs, fit-check table,
shield height by clay, C5 and antenna, device-1 log codes). The fit sheets
show the socket bodies, free support bands, the C5 clamp envelope and the
microSD corridor. BRINGUP gains the installation sequence (flex bridge
checks, harness polarity, tail voltages, staged boot), realistic bench
stages for the FPGA link, installed probing, and fixes (U10.3 clock, R410
1 k). Docs now state that Q20 blocks a reversed feed only on the bench, that
arm B carries unfused console 3.3 V, the tap fuse part (0251002.MXL), the
LBA28 limit and the watchdog rule. Stale "no further teardown" statements
are corrected.

Regenerated: schematic, ERC, netlist, integration and parts audits, BOM,
assembly drafts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
Parts:
- U21, U22: value TPS62162 3.3V 1A -> TPS62172 3.3V 0.5A; MPN TPS62162DSGR -> TPS62172DSGR
Changed lines of the file:
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@@
 (symbol (lib_id "KUI_G1:U21") (at 157.48 97.79 0) (unit 1) (in_bom yes) (on_board yes) (dnp no)
  (property "Reference" "U21" (at 157.48 85.09 0) (effects (font (size 1.0 1.0))))
- (property "Value" "TPS62162 3.3V 1A" (at 157.48 87.63 0) (effects (font (size 1.0 1.0))))
+ (property "Value" "TPS62172 3.3V 0.5A" (at 157.48 87.63 0) (effects (font (size 1.0 1.0))))
  (property "Footprint" "KUI_Footprints:TI_DSG0008A" (at 157.48 97.79 0) (effects (font (size 1.0 1.0)) hide))
- (property "Datasheet" "https://www.ti.com/lit/ds/symlink/tps62162.pdf" (at 157.48 97.79 0) (effects (font (size 1.0 1.0)) hide))
- (property "MPN" "TPS62162DSGR" (at 157.48 97.79 0) (effects (font (size 1.0 1.0)) hide))
+ (property "Datasheet" "https://www.ti.com/lit/ds/symlink/tps62170.pdf" (at 157.48 97.79 0) (effects (font (size 1.0 1.0)) hide))
+ (property "MPN" "TPS62172DSGR" (at 157.48 97.79 0) (effects (font (size 1.0 1.0)) hide))
  (property "LCSC" "" (at 157.48 97.79 0) (effects (font (size 1.0 1.0)) hide))
  (property "Variant" "BASE" (at 157.48 97.79 0) (effects (font (size 1.0 1.0)) hide))
@@
 (symbol (lib_id "KUI_G1:U22") (at 157.48 214.63 0) (unit 1) (in_bom yes) (on_board yes) (dnp no)
  (property "Reference" "U22" (at 157.48 201.93 0) (effects (font (size 1.0 1.0))))
- (property "Value" "TPS62162 3.3V 1A" (at 157.48 204.47 0) (effects (font (size 1.0 1.0))))
+ (property "Value" "TPS62172 3.3V 0.5A" (at 157.48 204.47 0) (effects (font (size 1.0 1.0))))
  (property "Footprint" "KUI_Footprints:TI_DSG0008A" (at 157.48 214.63 0) (effects (font (size 1.0 1.0)) hide))
- (property "Datasheet" "https://www.ti.com/lit/ds/symlink/tps62162.pdf" (at 157.48 214.63 0) (effects (font (size 1.0 1.0)) hide))
- (property "MPN" "TPS62162DSGR" (at 157.48 214.63 0) (effects (font (size 1.0 1.0)) hide))
+ (property "Datasheet" "https://www.ti.com/lit/ds/symlink/tps62170.pdf" (at 157.48 214.63 0) (effects (font (size 1.0 1.0)) hide))
+ (property "MPN" "TPS62172DSGR" (at 157.48 214.63 0) (effects (font (size 1.0 1.0)) hide))
  (property "LCSC" "" (at 157.48 214.63 0) (effects (font (size 1.0 1.0)) hide))
  (property "Variant" "BASE" (at 157.48 214.63 0) (effects (font (size 1.0 1.0)) hide))
