File: hardware/g1-sd-wifi/controller/controller-3.kicad_sch (KiCad schematic)
At the start: 20 parts, among them J202 RP USB service pads, J203 RP SWD/reset/boot pads, J204 C5 direct UART recovery pads, K201 C5 removable compression cont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, K202 C5 removable compression cont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, K203 C5 removable compression cont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, K204 C5 removable compression cont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, K205 C5 removable compression cont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, K206 C5 removable compression cont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, K207 C5 removable compression cont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, K208 C5 removable compression cont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, K209 C5 removable compression cont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, K210 C5 removable compression cont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, K211 C5 removable compression cont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, K212 C5 removable compression cont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, K213 C5 removable compression cont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, K214 C5 removable compression cont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, K215 C5 removable compression cont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, K216 C5 removable compression cont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

Commit message: G1 carrier: wire the FPGA JTAG and PROGRAMN to the RP2350
U201 GPIO21 (TMS), GPIO22 (TCK), GPIO29 (TDI), GPIO30 (TDO) and GPIO28
(PROGRAMN) now reach U10 through 220-ohm series resistors R2044-R2048, so
the controller can configure the FPGA in-system and a J10 cable is needed
only until RP firmware exists. FPGA_DONE is not wired: the JTAG status
register reports it, and GPIO27 could only leave the package between
C2009's pads and past the crystal trace.

Routing starts from the fedc570 board and is replayed by
tools/rp_fpga_jtag_2026_10_17.sh: explicit U201 and U10 escapes, the gap
closer with F.Cu kept out of the 12-MHz crystal circuit and rip-up limited
to slow nets, two shallow junctions tidied (tools/edit_tracks.py), then
DRC with schematic parity (0 violations, 0 unconnected, 0 parity) and a
comparison with fedc570 (tools/check_preservation.py): every footprint,
zone and drawing unchanged; the only removed or shortened copper is on the
five lifted slow nets (USB_VBUS_SENSE, LINK_A1, USB_SERVICE_VBUS,
C5_PWR_EN, PWR_UPSTREAM_OK), which are rerouted.

fpga/bridge.lpf pins SYSCONFIG JTAG_PORT=ENABLE SDM_PORT=PROGRAMN_DONE_INITN.
design/blocks/controller.json records the firmware rules: configure only
inside a session with BRIDGE_ARM and FPGA_RESETn low and no G1 session
active, PROGRAMN open-drain, SAMPLE/PRELOAD all ones before ISC_ENABLE or
ISC_ENABLE_X, never EXTEST or CLAMP.

The resistor's LCSC code (C112291) comes from a search index; the parts
list marks it catalog_identity_search_index_only_assembly_pending until the
owner confirms it on lcsc.com and JLCPCB. Schematics, netlist, ERC, audits,
BOM/CPL, assembly drafts, fit PDFs, power-copper check, review evidence,
review-only package (now 2026-10-17) and preflight are regenerated. The
owner reviews in review-evidence.json are bound to the old hashes and must
be repeated.

The board diff (about 11,100 lines added, 3,000 removed) is the 821 new
tracks and vias, the five resistors and two refilled zones;
desig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
Parts:
- added R2044: 220, KUI_Footprints:R_0402_1005Metric, symbol KUI_G1:R2044
- added R2045: 220, KUI_Footprints:R_0402_1005Metric, symbol KUI_G1:R2045
- added R2046: 220, KUI_Footprints:R_0402_1005Metric, symbol KUI_G1:R2046
- added R2047: 220, KUI_Footprints:R_0402_1005Metric, symbol KUI_G1:R2047
- added R2048: 220, KUI_Footprints:R_0402_1005Metric, symbol KUI_G1:R2048
Connections:
- new net FPGA_PROGRAMn: R2048.2
- new net FPGA_PROGRAMn_MCU: R2048.1
- new net FPGA_TCK: R2044.2
- new net FPGA_TCK_MCU: R2044.1
- new net FPGA_TDI: R2046.2
- new net FPGA_TDI_MCU: R2046.1
- new net FPGA_TDO: R2047.2
- new net FPGA_TDO_MCU: R2047.1
- new net FPGA_TMS: R2045.2
- new net FPGA_TMS_MCU: R2045.1
Changed lines of the file:
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@@
  (wire (pts (xy 151.13 146.05) (xy 148.59 146.05)) (stroke (width 0) (type default)))
 (global_label "C5_ENn" (shape bidirectional) (at 148.59 146.05 0) (effects (font (size 0.85 0.85)) (justify right)))
+(symbol (lib_id "KUI_G1:R2044") (at 157.48 163.83 0) (unit 1) (in_bom yes) (on_board yes) (dnp no)
+ (property "Reference" "R2044" (at 157.48 156.21 0) (effects (font (size 1.0 1.0))))
+ (property "Value" "220" (at 157.48 158.75 0) (effects (font (size 1.0 1.0))))
+ (property "Footprint" "KUI_Footprints:R_0402_1005Metric" (at 157.48 163.83 0) (effects (font (size 1.0 1.0)) hide))
+ (property "Datasheet" "https://www.latticesemi.com/view_document?document_id=39085" (at 157.48 163.83 0) (effects (font (size 1.0 1.0)) hide))
+ (property "MPN" "RC0402FR-07220RL" (at 157.48 163.83 0) (effects (font (size 1.0 1.0)) hide))
+ (property "LCSC" "" (at 157.48 163.83 0) (effects (font (size 1.0 1.0)) hide))
+ (property "Variant" "BASE" (at 157.48 163.83 0) (effects (font (size 1.0 1.0)) hide))
+ (pin "1")
+ (pin "2")
+ (instances (project "KUI-G1-Bridge-RevA" (path "/8477501f-fac0-5337-89a1-fc3585ab7e6e/d5fa38d4-5582-5002-94de-d2722d83a9a5" (reference "R2044") (unit 1)))) )
+ (wire (pts (xy 151.13 163.83) (xy 148.59 163.83)) (stroke (width 0) (type default)))
+(global_label "FPGA_TCK_MCU" (shape bidirectional) (at 148.59 163.83 0) (effects (font (size 0.85 0.85)) (justify right)))
+ (wire (pts (xy 163.83 163.83) (xy 166.37 163.83)) (stroke (width 0) (type default)))
+(global_label "FPGA_TCK" (shape bidirectional) (at 166.37 163.83 180) (effects (font (size 0.85 0.85)) (justify left)))
+(symbol (lib_id "KUI_G1:R2045") (at 157.48 181.61 0) (unit 1) (in_bom yes) (on_board yes) (dnp no)
+ (property "Reference" "R2045" (at 157.48 173.99 0) (effects (font (size 1.0 1.0))))
+ (property "Value" "220" (at 157.48 176.53 0) (effects (font (size 1.0 1.0))))
+ (property "Footprint" "KUI_Footprints:R_0402_1005Metric" (at 157.48 181.61 0) (effects (font (size 1.0 1.0)) hide))
+ (property "Datasheet" "https://www.latticesemi.com/view_document?document_id=39085" (at 157.48 181.61 0) (effects (font (size 1.0 1.0)) hide))
+ (property "MPN" "RC0402FR-07220RL" (at 157.48 181.61 0) (effects (font (size 1.0 1.0)) hide))
+ (property "LCSC" "" (at 157.48 181.61 0) (effects (font (size 1.0 1.0)) hide))
+ (property "Variant" "BASE" (at 157.48 181.61 0) (effects (font (size 1.0 1.0)) hide))
+ (pin "1")
+ (pin "2")
+ (instances (project "KUI-G1-Bridge-RevA" (path "/8477501f-fac0-5337-89a1-fc3585ab7e6e/d5fa38d4-5582-5002-94de-d2722d83a9a5" (reference "R2045") (unit 1)))) )
+ (wire (pts (xy 151.13 181.61) (xy 148.59 181.61)) (stroke (width 0) (type default)))
+(global_label "FPGA_TMS_MCU" (shape bidirectional) (at 148.59 181.61 0) (effects (font (size 0.85 0.85)) (justify right)))
+ (wire (pts (xy 163.83 181.61) (xy 166.37 181.61)) (stroke (width 0) (type default)))
+(global_label "FPGA_TMS" (shape bidirectional) (at 166.37 181.61 180) (effects (font (size 0.85 0.85)) (justify left)))
+(symbol (lib_id "KUI_G1:R2046") (at 157.48 199.39 0) (unit 1) (in_bom yes) (on_board yes) (dnp no)
+ (property "Reference" "R2046" (at 157.48 191.77 0) (effects (font (size 1.0 1.0))))
+ (property "Value" "220" (at 157.48 194.31 0) (effects (font (size 1.0 1.0))))
+ (property "Footprint" "KUI_Footprints:R_0402_1005Metric" (at 157.48 199.39 0) (effects (font (size 1.0 1.0)) hide))
+ (property "Datasheet" "https://www.latticesemi.com/view_document?document_id=39085" (at 157.48 199.39 0) (effects (font (size 1.0 1.0)) hide))
+ (property "MPN" "RC0402FR-07220RL" (at 157.48 199.39 0) (effects (font (size 1.0 1.0)) hide))
+ (property "LCSC" "" (at 157.48 199.39 0) (effects (font (size 1.0 1.0)) hide))
+ (property "Variant" "BASE" (at 157.48 199.39 0) (effects (font (size 1.0 1.0)) hide))
+ (pin "1")
+ (pin "2")
+ (instances (project "KUI-G1-Bridge-RevA" (path "/8477501f-fac0-5337-89a1-fc3585ab7e6e/d5fa38d4-5582-5002-94de-d2722d83a9a5" (reference "R2046") (unit 1)))) )
+ (wire (pts (xy 151.13 199.39) (xy 148.59 199.39)) (stroke (width 0) (type default)))
+(global_label "FPGA_TDI_MCU" (shape bidirectional) (at 148.59 199.39 0) (effects (font (size 0.85 0.85)) (justify right)))
+ (wire (pts (xy 163.83 199.39) (xy 166.37 199.39)) (stroke (width 0) (type default)))
+(global_label "FPGA_TDI" (shape bidirectional) (at 166.37 199.39 180) (effects (font (size 0.85 0.85)) (justify left)))
+(symbol (lib_id "KUI_G1:R2047") (at 157.48 217.17 0) (unit 1) (in_bom yes) (on_board yes) (dnp no)
+ (property "Reference" "R2047" (at 157.48 209.55 0) (effects (font (size 1.0 1.0))))
+ (property "Value" "220" (at 157.48 212.09 0) (effects (font (size 1.0 1.0))))
+ (property "Footprint" "KUI_Footprints:R_0402_1005Metric" (at 157.48 217.17 0) (effects (font (size 1.0 1.0)) hide))
+ (property "Datasheet" "https://www.latticesemi.com/view_document?document_id=39085" (at 157.48 217.17 0) (effects (font (size 1.0 1.0)) hide))
+ (property "MPN" "RC0402FR-07220RL" (at 157.48 217.17 0) (effects (font (size 1.0 1.0)) hide))
+ (property "LCSC" "" (at 157.48 217.17 0) (effects (font (size 1.0 1.0)) hide))
+ (property "Variant" "BASE" (at 157.48 217.17 0) (effects (font (size 1.0 1.0)) hide))
+ (pin "1")
+ (pin "2")
+ (instances (project "KUI-G1-Bridge-RevA" (path "/8477501f-fac0-5337-89a1-fc3585ab7e6e/d5fa38d4-5582-5002-94de-d2722d83a9a5" (reference "R2047") (unit 1)))) )
+ (wire (pts (xy 151.13 217.17) (xy 148.59 217.17)) (stroke (width 0) (type default)))
+(global_label "FPGA_TDO_MCU" (shape bidirectional) (at 148.59 217.17 0) (effects (font (size 0.85 0.85)) (justify right)))
+ (wire (pts (xy 163.83 217.17) (xy 166.37 217.17)) (stroke (width 0) (type default)))
+(global_label "FPGA_TDO" (shape bidirectional) (at 166.37 217.17 180) (effects (font (size 0.85 0.85)) (justify left)))
+(symbol (lib_id "KUI_G1:R2048") (at 157.48 234.95 0) (unit 1) (in_bom yes) (on_board yes) (dnp no)
+ (property "Reference" "R2048" (at 157.48 227.33 0) (effects (font (size 1.0 1.0))))
+ (property "Value" "220" (at 157.48 229.87 0) (effects (font (size 1.0 1.0))))
+ (property "Footprint" "KUI_Footprints:R_0402_1005Metric" (at 157.48 234.95 0) (effects (font (size 1.0 1.0)) hide))
+ (property "Datasheet" "https://www.latticesemi.com/view_document?document_id=39085" (at 157.48 234.95 0) (effects (font (size 1.0 1.0)) hide))
+ (property "MPN" "RC0402FR-07220RL" (at 157.48 234.95 0) (effects (font (size 1.0 1.0)) hide))
+ (property "LCSC" "" (at 157.48 234.95 0) (effects (font (size 1.0 1.0)) hide))
+ (property "Variant" "BASE" (at 157.48 234.95 0) (effects (font (size 1.0 1.0)) hide))
+ (pin "1")
+ (pin "2")
+ (instances (project "KUI-G1-Bridge-RevA" (path "/8477501f-fac0-5337-89a1-fc3585ab7e6e/d5fa38d4-5582-5002-94de-d2722d83a9a5" (reference "R2048") (unit 1)))) )
+ (wire (pts (xy 151.13 234.95) (xy 148.59 234.95)) (stroke (width 0) (type default)))
+(global_label "FPGA_PROGRAMn_MCU" (shape bidirectional) (at 148.59 234.95 0) (effects (font (size 0.85 0.85)) (justify right)))
+ (wire (pts (xy 163.83 234.95) (xy 166.37 234.95)) (stroke (width 0) (type default)))
+(global_label "FPGA_PROGRAMn" (shape bidirectional) (at 166.37 234.95 180) (effects (font (size 0.85 0.85)) (justify left)))
  (embedded_fonts no)
 )
