File: hardware/g1-sd-wifi/design/routing-checkpoint/finishing-wip.kicad_pcb (KiCad board)
At the start: 6 copper layers, 59 x 115 mm, 351 parts, among them J10 FPGA JTAG pogo pads, J20 5V/GND direct wire pads, J201 microSD push-pull 1.42mm, J202 RP USB service pads, J203 RP SWD/reset/boot pads, J204 C5 direct UART recovery pads, J40 FH12-14S-0.5SH(55), J41 FH12-6S-0.5SH(55), J50 FH12-20S-0.5SH(55), J51 FH12-20S-0.5SH(55), K201 C5 removable compression cont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, K202 C5 removable compression cont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, K203 C5 removable compression cont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, K204 C5 removable compression cont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, K205 C5 removable compression cont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, K206 C5 removable compression cont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, K207 C5 removable compression cont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, K208 C5 removable compression cont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, K209 C5 removable compression cont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, K210 C5 removable compression cont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, K211 C5 removable compression cont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, K212 C5 removable compression cont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, K213 C5 removable compression cont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, K214 C5 removable compression cont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, K215 C5 removable compression cont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, K216 C5 removable compression cont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, Q20 PMV48XP reverse polarity, Q201 C5 recovery pull-down, Q202 C5 recovery pull-down, U10 LCMXO2-2000HC-4TG100C, U20 TPS2116 automatic mux, U201 RP2350B, U202 16MiB boot NOR, U203 8MiB QSPI PSRAM, U204 C5 off-state isolation, U205 C5 off-state isolation, U207 SD4-bit DAT rail isolation, U208 SD CLK/CMD rail isolation, U209 SD enable/power-good NAND, U21 TPS62162 3.3V 1A, U22 TPS62162 3.3V 1A, U23 TPS3808G33DBVR, U24 TPS3808G33DBVR, U25 TPS3808G33DBVR, U26 TPS3808G01DBVR, U27 SN74LVC2G08DCUR, U28 SN74LVC2G08DCUR, U29 SN74LVC2G08DCUR, U30 SN74LVC1G11DBVR, U31 SN74LVC2G04DBVT, U32 SN74LVC1G32DBVR, U33 SN74LVC1G08DBVR, U34 SN74LVC1G08DBVR, U35 SN74LVC16T245, U36 SN74LVC244A host controls, U37 SN74LVC1G17 host RESETn, U38 SN74LVC1G125 qualified ATA_IN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, U39 SN74LVC1G125 qualified ATA_DM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, U40 MX29LV640ETTI-70G x8 / 4 x 2M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, U41 SN74LVC2G125 bank-domain buff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, U42 SN74LVC1G11 write-authorize A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, U43 SN74LVC1G04 write-block inver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, U44 SN74LVC1G332 NOR WE qualifier, U45 TLV803EB29 console-rail NOR r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, U70 SN74LVC1G07 open-drain IORDY, U71 TPS22919 Wi-Fi input switch, U72 SN74LVC1G32DBVR, U73 SN74LVC1G32DBVR, X10 50MHz 3.3V, X201 12MHz

Commit message: G1 finishing: 8 open; optional In4 plane hops in the gap closer
KUI_PLANE_HOPS=1 lets signal connections use In4.Cu (the +3V3_LOGIC
plane) at four times the price per cell, where the four signal layers
are full. In1 (ground reference) is never used and supply nets never
hop. ATA_DD12 took one 10.5 mm hop; native DRC with zones refilled
accepts it and no net lost its plane connection.

Co-Authored-By: Claude Opus 5.5 <noreply@anthropic.com>
Claude-Session: https://claude.ai/code/session_01Gp9EYc2r9fMpZ7V8WtfonZ
Routing:
- net ATA_DD12: track 38.3 -> 109.3 mm, vias 3 -> 6

Commit message: G1 finishing: 7 open (DRC 0, parity 0, supply check passing)
Co-Authored-By: Claude Opus 5.5 <noreply@anthropic.com>
Claude-Session: https://claude.ai/code/session_01Gp9EYc2r9fMpZ7V8WtfonZ
Routing:
- net C5_SCLK_MCU: track 29.0 -> 0.71 mm, vias 2 -> 0
- net SD_DETECTn: track 36.5 -> 56.8 mm, vias 3 -> 4
- net ATA_INTRQ: track 57.8 -> 76.7 mm, vias 1 -> 4
- net MCU_USB_DM: track 12.2 -> 0.29 mm, vias 3 -> 1
- net MCU_USB_DP: track 0.07 -> 8.61 mm, vias 0 -> 3
- net LINK_A0: track 8.60 -> 16.6 mm, vias 1 -> 2
- net ATA_DD6: track 81.5 -> 89.3 mm, vias 5 -> 8
- net SD_DAT2_MCU: track 0.83 -> 8.27 mm, vias 0 -> 2
- net ATA_DD9: track 85.8 -> 91.7 mm, vias 5 -> 6
- net SD_CLK_MCU: track 20.9 -> 26.6 mm, vias 2 -> 4
- net C5_IRQ_MCU: track 40.3 -> 45.6 mm, vias 4 -> 5
- net LINK_A1: track 35.4 -> 40.5 mm, vias 4 -> 3
- net SD_DAT3_MCU: track 5.05 -> 0.15 mm
- net LINK_WRn: track 18.5 -> 14.3 mm
- net SD_DAT1_MCU: track 5.41 -> 9.04 mm
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